File: Commodore-64/MONster64/MONster64.sch (KiCad schematic (older format))
At the start: 90 parts, among them J1 USB Power, J10 4pin Expansion, J11 3v3, J12 GND, J13 Conn_01x20, J2 SWD, J3 USB_B_Micro, J4 Hirose_DM3D-SF, J5 RJ45_Amphenol_RJMG1BD3B8K1ANR, J6 CLOCK_JUMPER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

Commit message: Add files via upload
Parts:
- R1: renamed from R9; value 22K -> 10R
- renumbered C5 to C10, C6 to C11, C7 to C12, C8 to C13, C9 to C14, C10 to C15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
Other:
- moved on the sheet: C27, C28, C29, C30, C31, C32, C33, C34, C35, C36, C37, C38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
