File: Commodore-64/MONster64/MONster64 - NetModule.kicad_pcb (KiCad board)
At the start: 4 copper layers, 46 x 27.8 mm, 32 parts, among them J11 3v3, J12 GND, J13 Conn_01x20, J5 RJ45_Amphenol_RJMG1BD3B8K1ANR, U4 DP83822IFRHB, Y1 Crystal

Commit message: Add files via upload
Parts:
- moved C31 66.8 mm to (153.8, 90.9)
- moved C30 66.7 mm to (153.8, 92.9)
- moved C37 60.3 mm to (153.8, 98.8)
- moved C33 60.3 mm to (153.8, 85.0)
- moved C32 60.1 mm to (153.8, 87.0)
- moved C40 58.0 mm to (153.8, 96.8)
- moved C36 54.2 mm to (145.1, 94.6), turned to 270 degrees
- moved C39 51.2 mm to (143.1, 94.6), turned to 270 degrees
- moved R10 8.72 mm to (153.8, 89.0), turned to 180 degrees
- moved R12 6.64 mm to (153.8, 102.7), turned to 0 degrees
- moved R13 4.47 mm to (153.8, 100.8), turned to 180 degrees
- moved R14 4.40 mm to (141.2, 94.6)
- moved R17 3.92 mm to (139.2, 94.6), turned to 270 degrees
- moved R15 2.65 mm to (153.8, 94.9), turned to 180 degrees
- moved R16 0.51 mm to (137.2, 94.6)
- renumbered C21 to C27, C22 to C28, C23 to C29, C24 to C30, C25 to C31, C26 to C32, C27 to C33, C28 to C34, C29 to C35, C30 to C36, C31 to C37, C32 to C38, C33 to C39, C34 to C40, C35 to C41, C36 to C42, C37 to C43, C38 to C44, J13 to J12, J5 to J13, J11 to J7, J12 to J8, R12 to R10, R13 to R11, R14 to R12, R15 to R13, R16 to R14, R17 to R15, R7 to R16, R8 to R17
Routing:
- net GND: track 16.3 -> 102.6 mm, vias 7 -> 11
- net /ETH_TX_EN: track 10.8 -> 54.5 mm, vias 0 -> 1
- net /ETH_RX_D3: track 7.05 -> 50.7 mm, vias 0 -> 1
- net /ETH_RX_D2: track 8.64 -> 51.2 mm, vias 0 -> 1
- net /ETH_RX_D0: track 12.4 -> 54.6 mm, vias 0 -> 1
- net Net-(J13-PadR3): track 0.00 -> 41.3 mm, vias 0 -> 2
- net Net-(J13-PadL3): track 5.25 -> 43.3 mm, vias 1 -> 3
- net /ETH_RX_D1: track 16.1 -> 53.3 mm, vias 0 -> 1
- net /ETH_TX_D0: track 4.59 -> 41.7 mm, vias 0 -> 1
- net /ETH_COL: track 14.0 -> 50.5 mm
- net /ETH_RX_ER: track 17.6 -> 49.2 mm, vias 1 -> 2
- net /ETH_TX_D1: track 9.15 -> 40.7 mm, vias 0 -> 2
- net Net-(J13-PadR1): track 0.00 -> 29.6 mm, vias 0 -> 2
- net /ETH_TX_CLK: track 6.23 -> 35.0 mm
- net /ETH_RX_DV: track 14.1 -> 41.4 mm
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- added copper zone on In3.Cu, net GND
Other:
- board size 46 x 27.8 mm -> 46 x 28.3 mm
- copper layers 4 -> 6
