File: Commodore-64/MONster64/MONster64.kicad_pcb (KiCad board)
At the start: 2 copper layers, 57.9 x 67.9 mm, 58 parts, among them J1 USB Power, J10 4pin Expansion, J2 SWD, J3 USB_B_Micro, J4 Hirose_DM3D-SF, J6 CLOCK_JUMPER, J7 3v3, J8 GND, J9 Conn_01x20, Q1 BC846BLT1G, SW1 Reset, SW2 Menu, SW3 Special, U1 STM32H753VIT6, U2 TXS0108EQPWRQ1, U3 W25M02GWZEIG, X1 DSC1001

Commit message: added some jumper labels to the front silkscreen
Other:
- board text added: "BOOT0 +3V3 GND SWDIO SWCLK"
- board text added: "DOT/8MHz"
- board text added: "USB5V"
Changed lines of the file:
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@@
   (general
     (thickness 1.6)
-    (drawings 10)
+    (drawings 13)
     (tracks 2167)
     (zones 0)
@@
     )
   )
+  (gr_text USB5V (at 100.7745 86.868 270) (layer F.SilkS)
+    (effects (font (size 1.5 1.5) (thickness 0.3)))
+  )
+  (gr_text DOT/8MHz (at 95.885 107.2515) (layer F.SilkS)
+    (effects (font (size 1.3 1.3) (thickness 0.3)))
+  )
+  (gr_text "BOOT0\n+3V3\nGND\nSWDIO\nSWCLK" (at 90.1065 83.5025 270) (layer F.SilkS)
+    (effects (font (size 1.5 1.3) (thickness 0.3)) (justify left))
+  )
   (target plus (at 103.3145 85.852) (size 5) (width 0.1) (layer Edge.Cuts))

Commit message: Add files via upload
Parts:
- R1: renamed from R9; value 22K -> 10R
- renumbered C5 to C10, C6 to C11, C7 to C12, C8 to C13, C9 to C14, C10 to C15, C11 to C16, C12 to C17, C13 to C18, C14 to C19, C39 to C2, C15 to C20, C16 to C21, C17 to C22, C18 to C23, C19 to C24, C20 to C25, C44 to C26, C41 to C3, C2 to C4, C42 to C5, C40 to C6, C43 to C7, C3 to C8, C4 to C9, D2 to D1, D1 to D2, J3 to J10, J4 to J11, J6 to J2, J7 to J3, J10 to J4, J9 to J5, J8 to J6, J2 to J9, R1 to R2, R2 to R3, R3 to R4, R10 to R5, R11 to R6, R4 to R7, R5 to R8, R6 to R9

Commit message: Add files via upload
Other:
- board text added: "Menu"
- board text added: "Reset"
- board text added: "Special"
Changed lines of the file:
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@@
   (general
     (thickness 1.6)
-    (drawings 13)
+    (drawings 16)
     (tracks 2167)
     (zones 0)
@@
     )
   )
+  (gr_text Menu (at 91.948 75.1205 270) (layer F.SilkS)
+    (effects (font (size 1.5 1.5) (thickness 0.3)))
+  )
+  (gr_text Reset (at 109.982 80.0735) (layer F.SilkS)
+    (effects (font (size 1.5 1.5) (thickness 0.3)))
+  )
+  (gr_text Special (at 69.0245 75.7555 270) (layer F.SilkS)
+    (effects (font (size 1.5 1.5) (thickness 0.3)))
+  )
   (gr_text USB5V (at 100.7745 86.868 270) (layer F.SilkS)
     (effects (font (size 1.5 1.5) (thickness 0.3)))
@@
   (segment (start 76.968541 110.361843) (end 76.968541 111.379347) (width 0.295) (layer F.Cu) (net 6))
   (segment (start 79.643501 113.459999) (end 80.133801 113.459999) (width 0.295) (layer F.Cu) (net 6))
-  (segment (start 97.273 75.683) (end 98.1075 76.5175) (width 1.5) (layer B.Cu) (net 111))
-  (segment (start 93.98 75.683) (end 97.273 75.683) (width 1.5) (layer B.Cu) (net 111))
   (segment (start 107.581 88.422) (end 108.5515 88.422) (width 0.439) (layer F.Cu) (net 7))
   (segment (start 108.5515 88.422) (end 108.712 88.5825) (width 0.439) (layer F.Cu) (net 7))
@@
   (segment (start 86.869548 105.156) (end 86.869548 105.157548) (width 0.295) (layer B.Cu) (net 20))
   (segment (start 86.869548 105.157548) (end 87.5665 105.8545) (width 0.295) (layer B.Cu) (net 20))
-  (segment (start 68.277 75.438) (end 66.19 77.525) (width 1.5) (layer B.Cu) (net 114))
-  (segment (start 69.46 75.438) (end 68.277 75.438) (width 1.5) (layer B.Cu) (net 114))
-  (segment (start 66.19 77.525) (end 59.69 77.525) (width 1.5) (layer B.Cu) (net 114))
   (segment (start 101.505 126.9045) (end 101.505 125.96) (width 0.295) (layer F.Cu) (net 21))
   (segment (start 98.298 130.1115) (end 101.505 126.9045) (width 0.295) (layer F.Cu) (net 21))
@@
   (segment (start 93.80749 128.962902) (end 93.80749 125.78749) (width 0.295) (layer F.Cu) (net 66))
   (segment (start 91.134892 131.6355) (end 93.80749 128.962902) (width 0.295) (layer F.Cu) (net 66))
-  (segment (start 83.07201 123.11249) (end 81.92901 123.11249) (width 0.295) (layer F.Cu) (net 109))
-  (segment (start 83.13 123.11) (end 83.0745 123.11) (width 0.295) (layer F.Cu) (net 109))
-  (segment (start 83.0745 123.11) (end 83.07201 123.11249) (width 0.295) (layer F.Cu) (net 109))
-  (segment (start 81.92901 123.11249) (end 81.915 123.1265) (width 0.295) (layer F.Cu) (net 109))
-  (via (at 81.915 123.1265) (size 0.35) (drill 0.3) (layers F.Cu B.Cu) (net 109))
-  (segment (start 82.8585 123.1265) (end 83.185 122.8) (width 0.295) (layer B.Cu) (net 109))
-  (segment (start 81.915 123.1265) (end 82.8585 123.1265) (width 0.295) (layer B.Cu) (net 109))
-  (segment (start 95.758 127.127) (end 95.758 127.127) (width 0.295) (layer B.Cu) (net 110))
-  (via (at 95.758 127.127) (size 0.35) (drill 0.3) (layers F.Cu B.Cu) (net 110))
-  (segment (start 95.805 127.08) (end 95.758 127.127) (width 0.295) (layer F.Cu) (net 110))
-  (segment (start 95.805 125.785) (end 95.805 127.08) (width 0.295) (layer F.Cu) (net 110))
-  (segment (start 94.615 125.984) (end 95.758 127.127) (width 0.295) (layer B.Cu) (net 110))
-  (segment (start 94.615 124.85) (end 94.615 125.984) (width 0.295) (layer B.Cu) (net 110))
-  (segment (start 83.1215 77.525) (end 89.6215 77.525) (width 1.5) (layer B.Cu) (net 113))
-  (segment (start 80.218 77.525) (end 79.765 77.978) (width 1.5) (layer B.Cu) (net 113))
-  (segment (start 83.1215 77.525) (end 80.218 77.525) (width 1.5) (layer B.Cu) (net 113))
   (segment (start 73.146 115.57) (end 72.5805 116.1355) (width 0.295) (layer F.Cu) (net 67))
   (segment (start 74.041 115.57) (end 73.146 115.57) (width 0.295) (layer F.Cu) (net 67))
@@
   (segment (start 86.508852 104.013) (end 94.615 95.906852) (width 0.295) (layer F.Cu) (net 107))
   (segment (start 83.317698 105.283) (end 84.582 105.283) (width 0.295) (layer F.Cu) (net 107))
+  (segment (start 83.07201 123.11249) (end 81.92901 123.11249) (width 0.295) (layer F.Cu) (net 109))
+  (segment (start 83.13 123.11) (end 83.0745 123.11) (width 0.295) (layer F.Cu) (net 109))
+  (segment (start 83.0745 123.11) (end 83.07201 123.11249) (width 0.295) (layer F.Cu) (net 109))
+  (segment (start 81.92901 123.11249) (end 81.915 123.1265) (width 0.295) (layer F.Cu) (net 109))
+  (via (at 81.915 123.1265) (size 0.35) (drill 0.3) (layers F.Cu B.Cu) (net 109))
+  (segment (start 82.8585 123.1265) (end 83.185 122.8) (width 0.295) (layer B.Cu) (net 109))
+  (segment (start 81.915 123.1265) (end 82.8585 123.1265) (width 0.295) (layer B.Cu) (net 109))
+  (segment (start 95.758 127.127) (end 95.758 127.127) (width 0.295) (layer B.Cu) (net 110))
+  (via (at 95.758 127.127) (size 0.35) (drill 0.3) (layers F.Cu B.Cu) (net 110))
+  (segment (start 95.805 127.08) (end 95.758 127.127) (width 0.295) (layer F.Cu) (net 110))
+  (segment (start 95.805 125.785) (end 95.805 127.08) (width 0.295) (layer F.Cu) (net 110))
+  (segment (start 94.615 125.984) (end 95.758 127.127) (width 0.295) (layer B.Cu) (net 110))
+  (segment (start 94.615 124.85) (end 94.615 125.984) (width 0.295) (layer B.Cu) (net 110))
+  (segment (start 97.273 75.683) (end 98.1075 76.5175) (width 1.5) (layer B.Cu) (net 111))
+  (segment (start 93.98 75.683) (end 97.273 75.683) (width 1.5) (layer B.Cu) (net 111))
+  (segment (start 83.1215 77.525) (end 89.6215 77.525) (width 1.5) (layer B.Cu) (net 113))
+  (segment (start 80.218 77.525) (end 79.765 77.978) (width 1.5) (layer B.Cu) (net 113))
+  (segment (start 83.1215 77.525) (end 80.218 77.525) (width 1.5) (layer B.Cu) (net 113))
+  (segment (start 68.277 75.438) (end 66.19 77.525) (width 1.5) (layer B.Cu) (net 114))
+  (segment (start 69.46 75.438) (end 68.277 75.438) (width 1.5) (layer B.Cu) (net 114))
+  (segment (start 66.19 77.525) (end 59.69 77.525) (width 1.5) (layer B.Cu) (net 114))
   (zone (net 1) (net_name GND) (layer F.Cu) (hatch edge 0.508)
     (connect_pads (clearance 0.239))

Commit message: Changed over for 1v8 operation
- Level Translated DOTCLK for OSC_IN
- JTAG header requires 5v instead of 3v3 to power board
- NAND Flash memory directly connected instead of through a TXS0108
- Dual regulator to streamline power domains.
Parts:
- removed D1: MMSZ4678T1G 1v8, Diode_SMD:D_SOD-123
- removed LVO1: NCP1117LPST33T3G, Package_TO_SOT_SMD:SOT-223-3_TabPin2
- removed R1: 10R, Resistor_SMD:R_0805_2012Metric_Pad1.15x1.40mm_HandSolder
- removed U2: TXS0108EQPWRQ1, Package_SO:TSSOP-20_4.4x6.5mm_P0.65mm
- added U5: MIC5356-SGYMME, Package_SO:MSOP-8-1EP_3x3mm_P0.65mm_EP2.5x3mm_Mask1.73x2.36mm_ThermalVias, F.Cu at (66.2, 124.2)
- added U6: SN74LV1T34DCKR, Package_TO_SOT_SMD:SOT-353_SC-70-5, F.Cu at (77.5, 124.0)
- R7, R8, R9: value 510R -> 150R
- RN1, RN2: footprint Resistor_SMD:R_Array_Convex_4x1206 -> Resistor_SMD:R_Array_Concave_4x0603
- X1: value DSC1001 -> DSC1001BI2-008.0000
- moved C25 12.4 mm to (102.4, 112.8), turned to 180 degrees
- moved C7 9.37 mm to (66.4, 121.4), turned to 180 degrees
- moved C3 6.13 mm to (65.0, 113.7), turned to 180 degrees
- moved C5 5.84 mm to (73.0, 125.2)
- moved U3 3.89 mm to (71.2, 117.5), turned to 90 degrees
- moved C18 3.24 mm to (75.2, 125.2), turned to 270 degrees
- moved RN1 2.73 mm to (106.2, 124.5)
- moved C15 2.31 mm to (77.4, 125.2), turned to 270 degrees
- moved C10 1.31 mm to (80.3, 125.1), turned to 0 degrees
- moved RN2 0.76 mm to (110.6, 124.5)
- moved Q1 0.13 mm to (60.3, 114.2)
Connections:
- C10 pad 1: +3V3 -> +1V8
- C11 pad 1: +3V3 -> +1V8
- C12 pad 1: +3V3 -> +1V8
- C13 pad 1: +3V3 -> +1V8
- C14 pad 1: +3V3 -> +1V8
- C15 pad 1: +3V3 -> +1V8
- C16 pad 1: +3V3 -> +1V8
- C17 pad 1: +3V3 -> +1V8
- C18 pad 1: +3V3 -> +1V8
- C19 pad 1: +3V3 -> +1V8
- C6 pad 1: +3V3 -> +1V8
- C8 pad 1: +3V3 -> +1V8
- C9 pad 1: +3V3 -> +1V8
- J2 pad 1: /DOT -> /DOT_1V8
- J4 pad 6: +3V3 -> +1V8
- J9 pad 2: +3V3 -> +5V
- R4 pad 1: +3V3 -> +1V8
- SW2 pad 1: +3V3 -> +1V8
- SW3 pad 1: +3V3 -> +1V8
- U1 pad 100: +3V3 -> +1V8
- U1 pad 11: +3V3 -> +1V8
- U1 pad 20: +3V3 -> +1V8
- U1 pad 21: +3V3 -> +1V8
- U1 pad 27: +3V3 -> +1V8
- U1 pad 50: +3V3 -> +1V8
- U1 pad 6: +3V3 -> +1V8
- U1 pad 75: +3V3 -> +1V8
- U3 pad 1: Net-(U2-Pad7) -> /NF_~CS
- U3 pad 2: Net-(U2-Pad3) -> /NF_IO1
- U3 pad 3: Net-(U2-Pad4) -> /NF_IO2
- U3 pad 5: Net-(U2-Pad1) -> /NF_IO0
- U3 pad 6: Net-(U2-Pad6) -> /NF_CLK
- U3 pad 7: Net-(U2-Pad5) -> /NF_IO3
- X1 pad 4: +3V3 -> +1V8
Routing:
- net +1V8: track 26.0 -> 282.6 mm, vias 3 -> 16
- net +3V3: track 326.5 -> 182.4 mm, vias 22 -> 8
- net GND: track 449.9 -> 523.1 mm, vias 53 -> 67
- net /DOT_1V8: track 0.00 -> 38.5 mm, vias 0 -> 3
- net /DOT: track 52.1 -> 13.9 mm, vias 5 -> 2
- net /~RST: track 103.3 -> 77.7 mm, vias 4 -> 3
- net +5V: track 93.0 -> 111.2 mm, vias 3 -> 5
- net Net-(U2-Pad7): track 12.9 -> 0.00 mm, vias 2 -> 0
- net Net-(U2-Pad6): track 11.0 -> 0.00 mm, vias 2 -> 0
- net Net-(U2-Pad5): track 10.9 -> 0.00 mm
- net /NF_~CS: track 24.1 -> 34.9 mm
- net Net-(U2-Pad3): track 9.37 -> 0.00 mm, vias 2 -> 0
- net /NF_IO3: track 7.02 -> 16.2 mm, vias 0 -> 2
- net Net-(U2-Pad4): track 9.19 -> 0.00 mm, vias 2 -> 0
- net /NF_IO1: track 6.90 -> 15.8 mm
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Other:
- board text added: "BOOT0 +5V GND SWDIO SWCLK"
- board text removed: "BOOT0 +3V3 GND SWDIO SWCLK"

Commit message: Revert to 3v3
Still need to translate DOTclk
Parts:
- removed U5: MIC5356-SGYMME, Package_SO:MSOP-8-1EP_3x3mm_P0.65mm_EP2.5x3mm_Mask1.73x2.36mm_ThermalVias
- removed U6: SN74LV1T34DCKR, Package_TO_SOT_SMD:SOT-353_SC-70-5
- added D1: MMSZ4678T1G 1v8, Diode_SMD:D_SOD-123, F.Cu at (63.5, 114.3)
- added LVO1: NCP1117LPST33T3G, Package_TO_SOT_SMD:SOT-223-3_TabPin2, F.Cu at (64.1, 122.4)
- added R1: 10R, Resistor_SMD:R_0805_2012Metric_Pad1.15x1.40mm_HandSolder, B.Cu at (66.0, 122.6)
- added U2: TXS0108EQPWRQ1, Package_SO:TSSOP-20_4.4x6.5mm_P0.65mm, F.Cu at (73.7, 120.7)
- R7, R8, R9: value 150R -> 510R
- RN1, RN2: footprint Resistor_SMD:R_Array_Concave_4x0603 -> Resistor_SMD:R_Array_Convex_4x1206
- X1: value DSC1001BI2-008.0000 -> DSC1001
- moved C25 12.4 mm to (90.2, 114.9), turned to 90 degrees
- moved C7 9.37 mm to (75.6, 119.4), turned to 270 degrees
- moved C3 6.13 mm to (71.1, 113.0), turned to 270 degrees
- moved C5 5.84 mm to (73.0, 119.4)
- moved U3 3.89 mm to (70.5, 113.7), turned to 0 degrees
- moved C18 3.24 mm to (78.1, 123.8), turned to 90 degrees
- moved RN1 2.73 mm to (103.5, 124.5)
- moved C15 2.31 mm to (75.6, 123.8), turned to 90 degrees
- moved C10 1.31 mm to (80.6, 123.8), turned to 90 degrees
- moved RN2 0.76 mm to (109.9, 124.5)
- moved Q1 0.13 mm to (60.3, 114.3)
Connections:
- C10 pad 1: +1V8 -> +3V3
- C11 pad 1: +1V8 -> +3V3
- C12 pad 1: +1V8 -> +3V3
- C13 pad 1: +1V8 -> +3V3
- C14 pad 1: +1V8 -> +3V3
- C15 pad 1: +1V8 -> +3V3
- C16 pad 1: +1V8 -> +3V3
- C17 pad 1: +1V8 -> +3V3
- C18 pad 1: +1V8 -> +3V3
- C19 pad 1: +1V8 -> +3V3
- C6 pad 1: +1V8 -> +3V3
- C8 pad 1: +1V8 -> +3V3
- C9 pad 1: +1V8 -> +3V3
- J2 pad 1: /DOT_1V8 -> /DOT
- J4 pad 6: +1V8 -> +3V3
- J9 pad 2: +5V -> +3V3
- R4 pad 1: +1V8 -> +3V3
- SW2 pad 1: +1V8 -> +3V3
- SW3 pad 1: +1V8 -> +3V3
- U1 pad 100: +1V8 -> +3V3
- U1 pad 11: +1V8 -> +3V3
- U1 pad 20: +1V8 -> +3V3
- U1 pad 21: +1V8 -> +3V3
- U1 pad 27: +1V8 -> +3V3
- U1 pad 50: +1V8 -> +3V3
- U1 pad 6: +1V8 -> +3V3
- U1 pad 75: +1V8 -> +3V3
- U3 pad 1: /NF_~CS -> Net-(U2-Pad7)
- U3 pad 2: /NF_IO1 -> Net-(U2-Pad3)
- U3 pad 3: /NF_IO2 -> Net-(U2-Pad4)
- U3 pad 5: /NF_IO0 -> Net-(U2-Pad1)
- U3 pad 6: /NF_CLK -> Net-(U2-Pad6)
- U3 pad 7: /NF_IO3 -> Net-(U2-Pad5)
- X1 pad 4: +1V8 -> +3V3
Routing:
- net +1V8: track 282.6 -> 26.0 mm, vias 16 -> 3
- net +3V3: track 182.4 -> 326.5 mm, vias 8 -> 22
- net GND: track 523.1 -> 449.9 mm, vias 67 -> 53
- net /DOT_1V8: track 38.5 -> 0.00 mm, vias 3 -> 0
- net /DOT: track 13.9 -> 52.1 mm, vias 2 -> 5
- net /~RST: track 77.7 -> 103.3 mm, vias 3 -> 4
- net +5V: track 111.2 -> 93.0 mm, vias 5 -> 3
- net Net-(U2-Pad7): track 0.00 -> 12.9 mm, vias 0 -> 2
- net Net-(U2-Pad6): track 0.00 -> 11.0 mm, vias 0 -> 2
- net Net-(U2-Pad5): track 0.00 -> 10.9 mm
- net /NF_~CS: track 34.9 -> 24.1 mm
- net Net-(U2-Pad3): track 0.00 -> 9.37 mm, vias 0 -> 2
- net /NF_IO3: track 16.2 -> 7.02 mm, vias 2 -> 0
- net Net-(U2-Pad4): track 0.00 -> 9.19 mm, vias 0 -> 2
- net /NF_IO1: track 15.8 -> 6.90 mm
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Other:
- board text added: "BOOT0 +3V3 GND SWDIO SWCLK"
- board text removed: "BOOT0 +5V GND SWDIO SWCLK"

Commit message: Add files via upload
Parts:
- removed D1: MMSZ4678T1G 1v8, Diode_SMD:D_SOD-123
- removed LVO1: NCP1117LPST33T3G, Package_TO_SOT_SMD:SOT-223-3_TabPin2
- removed R1: 10R, Resistor_SMD:R_0805_2012Metric_Pad1.15x1.40mm_HandSolder
- added C45: 100n, Capacitor_SMD:C_0805_2012Metric_Pad1.15x1.40mm_HandSolder, B.Cu at (68.5, 125.5)
- added U5: SN74AUP1T34DCK, Package_TO_SOT_SMD:SOT-353_SC-70-5, F.Cu at (67.6, 125.3)
- added U6: MIC5356-SGYMME, Package_SO:MSOP-8-1EP_3x3mm_P0.65mm_EP2.5x3mm_Mask1.73x2.36mm_ThermalVias, F.Cu at (63.8, 120.2)
- moved C4 2.10 mm to (59.8, 124.1)
- moved C1 1.99 mm to (59.8, 121.8)
- moved C8 1.71 mm to (59.8, 119.6)
- moved C9 1.66 mm to (59.8, 117.3)
Connections:
- J2 pad 1: /DOT -> /DOT_3v3
- J9 pad 2: +3V3 -> +5V
Routing:
- net /DOT_3v3: track 0.00 -> 51.3 mm, vias 0 -> 3
- net /DOT: track 52.1 -> 16.5 mm, vias 5 -> 2
- net +5V: track 93.0 -> 110.7 mm, vias 3 -> 8
- net GND: track 449.9 -> 464.0 mm, vias 53 -> 52
- net +1V8: track 26.0 -> 20.2 mm, vias 3 -> 2
- net /~RESET: track 23.1 -> 27.1 mm
- net +3V3: track 326.5 -> 329.8 mm, vias 22 -> 18
- net /~LED: track 39.6 -> 42.2 mm
Other:
- board text added: "BOOT0 +5V GND SWDIO SWCLK"
- board text removed: "BOOT0 +3V3 GND SWDIO SWCLK"

Commit message: Add files via upload
Parts:
- U1: value STM32H753VIT6 -> STM32H743VIT6
- moved U6 0.60 mm to (63.2, 120.0)
Connections:
- U6 pad 1: +3V3 -> +5V
- U6 pad 3: +5V -> Net-(U6-Pad3)
- U6 pad 4: +5V -> Net-(U6-Pad4)
- U6 pad 5: +5V -> Net-(U6-Pad5)
- U6 pad 6: +1V8 -> Net-(U6-Pad6)
- U6 pad 7: (no net) -> +1V8
- U6 pad 8: (no net) -> +3V3
Routing:
- net +3V3: track 329.8 -> 333.4 mm, vias 18 -> 19
- net +5V: track 110.7 -> 114.2 mm, vias 8 -> 7
- net /NF_CLK: track 12.6 -> 10.9 mm
- net GND: track 464.0 -> 465.5 mm
- net +1V8: track 20.2 -> 21.1 mm

Commit message: Add files via upload
Routing:
- net GND: track 465.5 -> 483.8 mm
Other:
- board text added: "480MHz ARM Cortex-M7 2MB Program Memory 1MB Data RAM 256MB NAND Flash RAM +MicroSD slot +100Mb Network Module"
- board text removed: "400MHz ARM Cortex-M7 2MB Program Memory 1MB Data RAM 256MB NAND Flash RAM +MicroSD slot +100Mb Network Module"
Changed lines of the file:
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@@
   (general
     (thickness 1.6)
-    (drawings 16)
-    (tracks 2222)
+    (drawings 18)
+    (tracks 2233)
     (zones 0)
     (modules 58)
@@
   (layers
     (0 F.Cu signal)
-    (31 B.Cu signal)
+    (31 B.Cu signal hide)
     (32 B.Adhes user hide)
     (33 F.Adhes user hide)
     (34 B.Paste user hide)
     (35 F.Paste user hide)
-    (36 B.SilkS user hide)
-    (37 F.SilkS user hide)
+    (36 B.SilkS user)
+    (37 F.SilkS user)
     (38 B.Mask user hide)
     (39 F.Mask user hide)
@@
     (45 Margin user hide)
     (46 B.CrtYd user hide)
-    (47 F.CrtYd user hide)
+    (47 F.CrtYd user)
     (48 B.Fab user hide)
-    (49 F.Fab user hide)
+    (49 F.Fab user)
   )
   (setup
-    (last_trace_width 1)
+    (last_trace_width 0.25)
     (user_trace_width 0.295)
     (user_trace_width 0.357)
@@
     (tags "MSOP SO")
     (attr smd)
-    (fp_text reference U6 (at 0 -2.45 90) (layer F.SilkS)
+    (fp_text reference U6 (at 0 -2.286 90) (layer F.SilkS)
       (effects (font (size 1 1) (thickness 0.15)))
     )
@@
     )
   )
+  (dimension 43.815 (width 0.15) (layer F.Fab)
+    (gr_text "43.815 mm" (at 119.537 117.475 270) (layer F.Fab)
+      (effects (font (size 1 1) (thickness 0.15)))
+    )
+    (feature1 (pts (xy 86.36 139.3825) (xy 118.823421 139.3825)))
+    (feature2 (pts (xy 86.36 95.5675) (xy 118.823421 95.5675)))
+    (crossbar (pts (xy 118.237 95.5675) (xy 118.237 139.3825)))
+    (arrow1a (pts (xy 118.237 139.3825) (xy 117.650579 138.255996)))
+    (arrow1b (pts (xy 118.237 139.3825) (xy 118.823421 138.255996)))
+    (arrow2a (pts (xy 118.237 95.5675) (xy 117.650579 96.694004)))
+    (arrow2b (pts (xy 118.237 95.5675) (xy 118.823421 96.694004)))
+  )
+  (dimension 67.895 (width 0.15) (layer F.Fab)
+    (gr_text "67.895 mm" (at 122.839 105.435 90) (layer F.Fab)
+      (effects (font (size 1.5 1.5) (thickness 0.15)))
+    )
+    (feature1 (pts (xy 115.316 71.4875) (xy 122.125421 71.4875)))
+    (feature2 (pts (xy 115.316 139.3825) (xy 122.125421 139.3825)))
+    (crossbar (pts (xy 121.539 139.3825) (xy 121.539 71.4875)))
+    (arrow1a (pts (xy 121.539 71.4875) (xy 122.125421 72.614004)))
+    (arrow1b (pts (xy 121.539 71.4875) (xy 120.952579 72.614004)))
+    (arrow2a (pts (xy 121.539 139.3825) (xy 122.125421 138.255996)))
+    (arrow2b (pts (xy 121.539 139.3825) (xy 120.952579 138.255996)))
+  )
   (gr_text Menu (at 91.948 75.1205 270) (layer F.SilkS)
     (effects (font (size 1.5 1.5) (thickness 0.3)))
@@
     (effects (font (size 2.25 5) (thickness 0.4)))
   )
-  (gr_text "400MHz ARM Cortex-M7\n2MB Program Memory\n1MB Data RAM\n256MB NAND Flash RAM\n+MicroSD slot\n+100Mb Network Module" (at 70.8025 94.9325) (layer F.SilkS)
+  (gr_text "480MHz ARM Cortex-M7\n2MB Program Memory\n1MB Data RAM\n256MB NAND Flash RAM\n+MicroSD slot\n+100Mb Network Module" (at 70.8025 94.9325) (layer F.SilkS)
     (effects (font (size 1.2 1.2) (thickness 0.15)))
   )
@@
   (segment (start 63.242 118.9555) (end 63.254 118.9555) (width 0.65) (layer B.Cu) (net 1))
   (segment (start 62.6825 119.515) (end 63.242 118.9555) (width 0.65) (layer B.Cu) (net 1))
+  (segment (start 61.6825 120.015) (end 63.1825 120.015) (width 0.25) (layer F.Cu) (net 1))
+  (segment (start 63.5 114.4905) (end 63.075736 114.4905) (width 0.25) (layer F.Cu) (net 1))
+  (segment (start 63.075736 114.4905) (end 61.742236 115.824) (width 0.25) (layer F.Cu) (net 1))
+  (segment (start 60.17149 118.50399) (end 61.6825 120.015) (width 0.25) (layer F.Cu) (net 1))
+  (segment (start 60.17149 116.730192) (end 60.17149 118.50399) (width 0.25) (layer F.Cu) (net 1))
+  (segment (start 61.742236 115.824) (end 61.077682 115.824) (width 0.25) (layer F.Cu) (net 1))
+  (segment (start 61.077682 115.824) (end 60.17149 116.730192) (width 0.25) (layer F.Cu) (net 1))
+  (segment (start 70.285736 122.584) (end 70.71 122.584) (width 0.25) (layer F.Cu) (net 1))
+  (segment (start 68.254295 122.584) (end 70.285736 122.584) (width 0.25) (layer F.Cu) (net 1))
+  (segment (start 65.685295 120.015) (end 68.254295 122.584) (width 0.25) (layer F.Cu) (net 1))
+  (segment (start 63.1825 120.015) (end 65.685295 120.015) (width 0.25) (layer F.Cu) (net 1))
   (segment (start 62.1665 131.1275) (end 62.1665 136.306002) (width 1.5) (layer F.Cu) (net 2))
   (segment (start 62.1665 131.1275) (end 64.262 133.223) (width 1.5) (layer F.Cu) (net 2))
