File: Commodore-64/MONster64/MONster64.kicad_pcb (KiCad board)
At the start: 2 copper layers, 57.9 x 67.9 mm, 58 parts, among them J1 USB Power, J10 USB_B_Micro, J11 Hirose_DM3D-SF, J2 CLOCK_JUMPER, J3 3v3, J4 4pin Expansion, J5 Conn_01x20, J6 GND, J9 SWD, Q1 BC846BLT1G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

Commit message: Add files via upload
Parts:
- RN1, RN2: footprint Resistor_SMD:R_Array_Convex_4x1206 -> Resistor_SMD:R_Array_Concave_4x0603
- U1: value STM32H743VIT6 -> STM32H753VIT6
- moved RN2 0.70 mm to (109.2, 124.4)
- moved RN1 0.45 mm to (103.1, 124.4)
Routing:
- net GND: track 483.8 -> 584.4 mm
- net /D7: track 6.68 -> 8.56 mm
- net /CD7: track 15.7 -> 16.5 mm
- net /D2: track 14.8 -> 15.6 mm
- net /CD3: track 12.0 -> 12.8 mm
- net /CD6: track 14.4 -> 15.1 mm
- net /D3: track 13.3 -> 13.9 mm
- net /D6: track 8.68 -> 9.22 mm
- net /CD2: track 11.5 -> 12.0 mm

Commit message: Add files via upload
Connections:
- U6 pad 4: Net-(U6-Pad4) -> +5V
- U6 pad 5: Net-(U6-Pad5) -> +5V
Routing:
- net +5V: track 114.2 -> 115.7 mm, vias 7 -> 9
Other:
- board text added: "JAYSTONIAN"
Changed lines of the file:
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@@
   (general
     (thickness 1.6)
-    (drawings 18)
-    (tracks 2290)
+    (drawings 20)
+    (tracks 2299)
     (zones 0)
     (modules 58)
-    (nets 121)
+    (nets 119)
   )
   (page A4)
   (layers
-    (0 F.Cu signal)
-    (31 B.Cu signal)
+    (0 F.Cu signal hide)
+    (31 B.Cu signal hide)
     (32 B.Adhes user hide)
     (33 F.Adhes user hide)
     (34 B.Paste user hide)
     (35 F.Paste user hide)
-    (36 B.SilkS user)
+    (36 B.SilkS user hide)
     (37 F.SilkS user)
     (38 B.Mask user hide)
@@
   )
   (setup
-    (last_trace_width 0.295)
+    (last_trace_width 0.25)
     (user_trace_width 0.295)
     (user_trace_width 0.357)
@@
   (net 116 "Net-(U5-Pad1)")
   (net 117 "Net-(U6-Pad3)")
-  (net 118 "Net-(U6-Pad4)")
-  (net 119 "Net-(U6-Pad5)")
-  (net 120 "Net-(U6-Pad6)")
+  (net 118 "Net-(U6-Pad6)")
   (net_class Default "This is the default net class."
     (clearance 0.2)
@@
     (add_net "Net-(U5-Pad1)")
     (add_net "Net-(U6-Pad3)")
-    (add_net "Net-(U6-Pad4)")
-    (add_net "Net-(U6-Pad5)")
     (add_net "Net-(U6-Pad6)")
     (add_net "Net-(X1-Pad1)")
@@
       (net 117 "Net-(U6-Pad3)"))
     (pad 4 smd roundrect (at -2.175 0.975 90) (size 1.35 0.35) (layers F.Cu F.Paste F.Mask) (roundrect_rratio 0.25)
-      (net 118 "Net-(U6-Pad4)"))
+      (net 2 +5V))
     (pad 5 smd roundrect (at 2.175 0.975 90) (size 1.35 0.35) (layers F.Cu F.Paste F.Mask) (roundrect_rratio 0.25)
-      (net 119 "Net-(U6-Pad5)"))
+      (net 2 +5V))
     (pad 6 smd roundrect (at 2.175 0.325 90) (size 1.35 0.35) (layers F.Cu F.Paste F.Mask) (roundrect_rratio 0.25)
-      (net 120 "Net-(U6-Pad6)"))
+      (net 118 "Net-(U6-Pad6)"))
     (pad 7 smd roundrect (at 2.175 -0.325 90) (size 1.35 0.35) (layers F.Cu F.Paste F.Mask) (roundrect_rratio 0.25)
       (net 73 +1V8))
@@
     )
   )
+  (target plus (at 106.3371 124.4092) (size 5) (width 0.1) (layer Edge.Cuts))
+  (gr_text JAYSTONIAN (at 85.6615 130.937) (layer B.SilkS)
+    (effects (font (size 2.25 5) (thickness 0.5)) (justify mirror))
+  )
   (dimension 43.815 (width 0.15) (layer F.Fab)
     (gr_text "43.815 mm" (at 119.537 117.475 270) (layer F.Fab)
@@
   (segment (start 60.7695 121.793) (end 60.8965 121.793) (width 1.5) (layer F.Cu) (net 2))
   (via (at 60.7695 121.793) (size 0.8) (drill 0.4) (layers F.Cu B.Cu) (net 2))
+  (segment (start 64.92875 117.50675) (end 64.92875 117.50675) (width 0.65) (layer B.Cu) (net 2))
+  (via (at 64.92875 117.50675) (size 0.8) (drill 0.4) (layers F.Cu B.Cu) (net 2))
+  (segment (start 64.92875 117.50675) (end 64.35725 117.50675) (width 0.439) (layer F.Cu) (net 2))
+  (segment (start 64.35725 117.64025) (end 64.1575 117.84) (width 0.295) (layer F.Cu) (net 2))
+  (segment (start 64.35725 117.50675) (end 64.35725 117.64025) (width 0.295) (layer F.Cu) (net 2))
+  (segment (start 64.373 122.3805) (end 64.373 122.3805) (width 1.5) (layer B.Cu) (net 2))
+  (via (at 64.5795 122.301) (size 0.8) (drill 0.4) (layers F.Cu B.Cu) (net 2))
+  (segment (start 64.2685 122.301) (end 64.1575 122.19) (width 0.295) (layer F.Cu) (net 2))
+  (segment (start 64.5795 122.301) (end 64.2685 122.301) (width 0.295) (layer F.Cu) (net 2))
   (segment (start 76.835 101.219) (end 77.851 100.203) (width 1.5) (layer B.Cu) (net 3))
   (segment (start 81.407 115.1255) (end 80.645 115.8875) (width 0.65) (layer B.Cu) (net 3))

Commit message: Add files via upload
Routing:
- net GND: track 584.4 -> 613.3 mm
- net +3V3: track 333.4 -> 331.8 mm
Changed lines of the file:
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@@
     (thickness 1.6)
     (drawings 20)
-    (tracks 2299)
+    (tracks 2310)
     (zones 0)
     (modules 58)
@@
   (page A4)
   (layers
-    (0 F.Cu signal hide)
-    (31 B.Cu signal hide)
+    (0 F.Cu signal)
+    (31 B.Cu signal)
     (32 B.Adhes user hide)
     (33 F.Adhes user hide)
@@
   )
   (setup
-    (last_trace_width 0.25)
+    (last_trace_width 1.5)
     (user_trace_width 0.295)
     (user_trace_width 0.357)
@@
     )
   )
-  (target plus (at 106.3371 124.4092) (size 5) (width 0.1) (layer Edge.Cuts))
+  (target plus (at 106.3371 124.3965) (size 5) (width 0.1) (layer Edge.Cuts))
   (gr_text JAYSTONIAN (at 85.6615 130.937) (layer B.SilkS)
     (effects (font (size 2.25 5) (thickness 0.5)) (justify mirror))
@@
     (arrow2b (pts (xy 122.682 139.3825) (xy 122.095579 138.255996)))
   )
+  (segment (start 112.7887 132.334) (end 112.0902 131.6355) (width 1.5) (layer B.Cu) (net 1))
+  (segment (start 114.0079 131.5593) (end 113.3094 132.2578) (width 1.5) (layer F.Cu) (net 1))
+  (segment (start 112.141 131.6863) (end 112.8395 132.3848) (width 1.5) (layer F.Cu) (net 1))
+  (segment (start 113.7158 130.1623) (end 113.0173 130.8608) (width 1.5) (layer F.Cu) (net 1))
+  (segment (start 58.8518 131.699) (end 59.5503 132.3975) (width 1.5) (layer F.Cu) (net 1))
   (segment (start 113.7285 122.1105) (end 113.7285 129.2225) (width 1) (layer F.Cu) (net 1))
   (segment (start 63.1905 119.372) (end 63.6905 118.872) (width 1.5) (layer B.Cu) (net 1))
@@
   (via (at 89.1667 103.5177) (size 0.8) (drill 0.4) (layers F.Cu B.Cu) (net 1))
   (via (at 89.6874 107.5182) (size 0.8) (drill 0.4) (layers F.Cu B.Cu) (net 1))
-  (via (at 106.3371 124.4092) (size 0.35) (drill 0.3) (layers F.Cu B.Cu) (net 1))
-  (via (at 108.7882 124.4219) (size 0.35) (drill 0.3) (layers F.Cu B.Cu) (net 1))
+  (via (at 106.3371 124.3965) (size 0.35) (drill 0.3) (layers F.Cu B.Cu) (net 1))
+  (via (at 108.7882 124.3965) (size 0.35) (drill 0.3) (layers F.Cu B.Cu) (net 1))
   (via (at 103.5431 124.4092) (size 0.35) (drill 0.3) (layers F.Cu B.Cu) (net 1))
   (via (at 101.6254 124.4092) (size 0.35) (drill 0.3) (layers F.Cu B.Cu) (net 1))
@@
   (segment (start 61.742236 115.824) (end 61.077682 115.824) (width 0.25) (layer F.Cu) (net 1))
   (segment (start 61.077682 115.824) (end 60.17149 116.730192) (width 0.25) (layer F.Cu) (net 1))
-  (segment (start 70.285736 122.584) (end 70.71 122.584) (width 0.25) (layer F.Cu) (net 1))
-  (segment (start 68.254295 122.584) (end 70.285736 122.584) (width 0.25) (layer F.Cu) (net 1))
-  (segment (start 65.685295 120.015) (end 68.254295 122.584) (width 0.25) (layer F.Cu) (net 1))
-  (segment (start 63.1825 120.015) (end 65.685295 120.015) (width 0.25) (layer F.Cu) (net 1))
   (segment (start 58.124991 122.450491) (end 58.36671 122.69221) (width 0.25) (layer F.Cu) (net 1))
   (segment (start 58.36671 122.69221) (end 58.36671 124.13229) (width 0.25) (layer F.Cu) (net 1))
@@
   (segment (start 66.2813 126.6952) (end 66.6115 126.365) (width 0.295) (layer F.Cu) (net 1))
   (segment (start 66.2813 131.318) (end 66.2813 126.6952) (width 0.295) (layer F.Cu) (net 1))
-  (segment (start 62.1665 131.1275) (end 62.1665 136.306002) (width 1.5) (layer F.Cu) (net 2))
+  (segment (start 64.6825 120.015) (end 63.1825 120.015) (width 1.5) (layer F.Cu) (net 1))
+  (segment (start 66.074204 120.015) (end 64.6825 120.015) (width 1.5) (layer F.Cu) (net 1))
+  (segment (start 68.643204 122.584) (end 66.074204 120.015) (width 0.8) (layer F.Cu) (net 1))
+  (segment (start 70.71 122.584) (end 68.643204 122.584) (width 0.8) (layer F.Cu) (net 1))
+  (segment (start 61.6825 120.015) (end 60.452 118.7845) (width 0.8) (layer F.Cu) (net 1))
+  (segment (start 60.452 118.7845) (end 61.1265 118.7845) (width 0.8) (layer F.Cu) (net 1))
+  (segment (start 61.1265 118.7845) (end 61.6585 119.3165) (width 0.8) (layer F.Cu) (net 1))
+  (segment (start 59.3217 125.0442) (end 59.3217 132.9309) (width 1.5) (layer B.Cu) (net 1))
+  (segment (start 113.5761 120.5992) (end 113.5761 133.5659) (width 1.5) (layer B.Cu) (net 1))
+  (segment (start 62.103 131.1021) (end 62.103 136.280602) (width 1.5) (layer F.Cu) (net 2))
   (segment (start 62.1665 131.1275) (end 64.262 133.223) (width 1.5) (layer F.Cu) (net 2))
   (segment (start 62.1665 131.1275) (end 62.103 131.064) (width 1.5) (layer F.Cu) (net 2))
@@
   (segment (start 62.103 118.30425) (end 62.103 117.93075) (width 0.357) (layer F.Cu) (net 3))
   (segment (start 62.0875 118.2215) (end 61.9125 118.0465) (width 0.357) (layer F.Cu) (net 3))
-  (segment (start 62.0325 117.2915) (end 61.7715 117.0305) (width 0.357) (layer F.Cu) (net 3))
-  (segment (start 61.7715 117.0305) (end 60.8965 117.0305) (width 0.357) (layer F.Cu) (net 3))
-  (segment (start 60.8965 117.0305) (end 60.8965 117.0305) (width 0.357) (layer F.Cu) (net 3))
-  (via (at 60.8965 117.0305) (size 0.8) (drill 0.4) (layers F.Cu B.Cu) (net 3))
-  (segment (start 61.462185 117.0305) (end 61.849 117.417315) (width 0.8) (layer F.Cu) (net 3))
-  (segment (start 60.8965 117.0305) (end 61.462185 117.0305) (width 0.8) (layer F.Cu) (net 3))
+  (via (at 61.087 117.348) (size 0.8) (drill 0.4) (layers F.Cu B.Cu) (net 3))
   (segment (start 61.849 117.417315) (end 61.849 117.7925) (width 0.8) (layer F.Cu) (net 3))
   (segment (start 60.7785 117.2845) (end 60.7785 119.5705) (width 1.5) (layer B.Cu) (net 3))
@@
   (segment (start 60.7785 119.897) (end 60.7785 117.2845) (width 1) (layer B.Cu) (net 3))
   (segment (start 61.27449 120.39299) (end 60.7785 119.897) (width 1) (layer B.Cu) (net 3))
+  (segment (start 61.779685 117.348) (end 61.849 117.417315) (width 0.8) (layer F.Cu) (net 3))
+  (segment (start 61.087 117.348) (end 61.779685 117.348) (width 0.8) (layer F.Cu) (net 3))
   (segment (start 106.553 77.525) (end 113.053 77.525) (width 1.5) (layer B.Cu) (net 4))
   (segment (start 106.345 77.733) (end 106.553 77.525) (width 1.5) (layer B.Cu) (net 4))
@@
   (segment (start 64.77 126.365) (end 64.77 126.365) (width 0.295) (layer F.Cu) (net 18))
   (via (at 64.77 126.365) (size 0.6) (drill 0.4) (layers F.Cu B.Cu) (net 18))
-  (segment (start 60.58 115.604387) (end 59.35449 116.829897) (width 0.295) (layer F.Cu) (net 18))
-  (segment (start 60.58 114.995) (end 60.58 115.604387) (width 0.295) (layer F.Cu) (net 18))
-  (segment (start 59.35449 116.829897) (end 59.35449 125.07699) (width 0.295) (layer F.Cu) (net 18))
-  (segment (start 61.325 114.3) (end 61.275 114.3) (width 0.295) (layer F.Cu) (net 18))
-  (segment (start 61.275 114.3) (end 60.58 114.995) (width 0.295) (layer F.Cu) (net 18))
-  (segment (start 59.35449 125.07699) (end 60.6425 126.365) (width 0.295) (layer F.Cu) (net 18))
   (segment (start 60.6425 126.365) (end 60.6425 126.365) (width 0.295) (layer F.Cu) (net 18))
   (via (at 60.6425 126.365) (size 0.6) (drill 0.4) (layers F.Cu B.Cu) (net 18))
   (segment (start 61.066764 126.365) (end 64.77 126.365) (width 0.295) (layer B.Cu) (net 18))
   (segment (start 60.6425 126.365) (end 61.066764 126.365) (width 0.295) (layer B.Cu) (net 18))
+  (segment (start 61.275 114.3) (end 61.325 114.3) (width 0.295) (layer F.Cu) (net 18))
+  (segment (start 60.58 114.995) (end 61.275 114.3) (width 0.295) (layer F.Cu) (net 18))
+  (segment (start 59.35449 116.47701) (end 59.817 116.0145) (width 0.295) (layer F.Cu) (net 18))
+  (segment (start 59.35449 125.07699) (end 59.35449 116.47701) (width 0.295) (layer F.Cu) (net 18))
+  (segment (start 60.6425 126.365) (end 59.35449 125.07699) (width 0.295) (layer F.Cu) (net 18))
+  (segment (start 60.036002 116.0145) (end 60.198 115.852502) (width 0.295) (layer F.Cu) (net 18))
+  (segment (start 59.817 116.0145) (end 60.036002 116.0145) (width 0.295) (layer F.Cu) (net 18))
+  (segment (start 60.198 115.852502) (end 60.198 115.5065) (width 0.295) (layer F.Cu) (net 18))
+  (segment (start 60.58 115.1245) (end 60.58 114.995) (width 0.295) (layer F.Cu) (net 18))
+  (segment (start 60.198 115.5065) (end 60.58 115.1245) (width 0.295) (layer F.Cu) (net 18))
   (segment (start 94.805 109.635) (end 94.805 110.435) (width 0.295) (layer F.Cu) (net 19))
   (segment (start 94.361 77.978) (end 94.361 77.978) (width 0.295) (layer F.Cu) (net 19))
