File: Commodore-64/c64-cpm-smd/c64-cpm-smd.kicad_pcb (KiCad board)
At the start: 2 copper layers, 57.9 x 48.9 mm, 53 parts, among them Q1 CMPTA94, U1 SN74LV74APWR, U10 SN74F283D, U11 SN74LV245APWR, U12 4K7, U13 Z80CPU-QFP, U14 SN74LV245APWR, U15 4K7, U16 74LVC3G06, U2 SN74LV04APWR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

Commit message: Add files via upload
Parts:
- U16: value 74LVC3G06 -> 74LVC3G06DP
- U3: value 74HCT367PW,118 -> SN74LV367APWR
Connections:
- U12 pad 1: +5V -> /A5
- U12 pad 10: (no net) -> +5V
- U12 pad 2: /A5 -> /A4
- U12 pad 3: /A4 -> /A3
- U12 pad 4: /A3 -> /A2
- U12 pad 5: /A2 -> +5V
- U15 pad 1: +5V -> /A13
- U15 pad 10: (no net) -> +5V
- U15 pad 2: /A13 -> /A12
- U15 pad 3: /A12 -> /A11
- U15 pad 4: /A11 -> /A10
- U15 pad 5: /A10 -> +5V
- U8 pad 1: +5V -> /D7
- U8 pad 10: (no net) -> +5V
- U8 pad 2: /D7 -> /D6
- U8 pad 3: /D6 -> /D5
- U8 pad 4: /D5 -> /D4
- U8 pad 5: /D4 -> +5V
Routing:
- net +5V: track 261.0 -> 284.2 mm, vias 22 -> 25
- net /A5: track 19.8 -> 21.8 mm
- net /A4: track 18.5 -> 19.7 mm
- net /A13: track 18.3 -> 19.4 mm
- net /D4: track 22.8 -> 23.9 mm
- net /A3: track 17.4 -> 18.2 mm
- net /D6: track 21.2 -> 22.0 mm
- net /A12: track 16.9 -> 17.6 mm
- net GND: vias 72 -> 68
