File: Commodore-64/c64-cpm-smd/c64-cpm-smd.sch (KiCad schematic (older format))
At the start: 53 parts, among them Q1 CMPTA94, U1 SN74LV74APWR, U10 SN74F283D, U11 SN74LV245APWR, U12 4K7, U13 Z80CPU-QFP, U14 SN74LV245APWR, U15 4K7, U16 74LVC3G06, U2 SN74LV04APWR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

Commit message: Add files via upload
Parts:
- removed U12, U15, U8: 4K7, Resistor_SMD:R_Array_Convex_5x1206, symbol Device:R_Network08_US
- added U12, U15, U8: 4K7, Resistor_SMD:R_Array_Convex_5x1206, symbol CPU2:R_Network08_US_YC358-TType
- C1: footprint Capacitor_Tantalum_SMD:CP_EIA-6032-28_Kemet-C_Pad2.25x2.35mm_HandSolder -> Capacitor_THT:CP_Radial_D6.3mm_P2.50mm
- U16: value 74LVC3G06 -> 74LVC3G06DP
- U3: value 74HCT367PW,118 -> SN74LV367APWR
Connections:
- net +5V: now also U12.10 (common), U12.5 (common), U15.10 (common), U15.5 (common), U8.10 (common), U8.5 (common)
- net A0: now also U12.6 (R5)
- net A1: now also U12.7 (R6)
- net A10: now also U15.4 (R4)
- net A11: now also U15.3 (R3)
- net A12: now also U15.2 (R2)
- net A13: now also U15.1 (R1)
- net A14: now also U15.8 (R7)
- net A15: now also U15.9 (R8)
- net A2: now also U12.4 (R4)
- net A3: now also U12.3 (R3)
- net A4: now also U12.2 (R2)
- net A5: now also U12.1 (R1)
- net A6: now also U12.8 (R7)
- net A7: now also U12.9 (R8)
- net A8: now also U15.6 (R5)
- net A9: now also U15.7 (R6)
- net D0: now also U8.6 (R5)
- net D1: now also U8.7 (R6)
- net D2: now also U8.8 (R7)
- net D3: now also U8.9 (R8)
- net D4: now also U8.4 (R4)
- net D5: now also U8.3 (R3)
- net D6: now also U8.2 (R2)
- net D7: now also U8.1 (R1)
Changed lines of the file:
@@
 P 13950 7450
 F 0 "U3" H 14100 8100 50  0000 C CNN
-F 1 "74HCT367PW,118" H 14150 8000 50  0000 C CNN
+F 1 "SN74LV367APWR" H 14150 8000 50  0000 C CNN
 F 2 "Package_SO:TSSOP-16_4.4x5mm_P0.65mm" H 13950 7450 50  0001 C CNN
 F 3 "http://www.ti.com/lit/gpn/sn74LS367" H 13950 7450 50  0001 C CNN
@@
 $Comp
 L 74xx:74LS74 U1
-U 3 1 5E69BE1C
-P 850 5750
-F 0 "U1" H 1080 5796 50  0000 L CNN
-F 1 "SN74LV74APWR" H 1080 5705 50  0000 L CNN
-F 2 "Package_SO:TSSOP-14_4.4x5mm_P0.65mm" H 850 5750 50  0001 C CNN
-F 3 "74xx/74hc_hct74.pdf" H 850 5750 50  0001 C CNN
-	3    850  5750
-	1    0    0    -1
-$EndComp
-$Comp
-L 74xx:74LS74 U1
 U 1 1 5E69BE22
 P 850 10350
@@
 F 0 "C1" H 3188 7246 50  0000 L CNN
 F 1 "47uF" H 3188 7155 50  0000 L CNN
-F 2 "Capacitor_Tantalum_SMD:CP_EIA-6032-28_Kemet-C_Pad2.25x2.35mm_HandSolder" H 3100 7200 50  0001 C CNN
+F 2 "Capacitor_THT:CP_Radial_D6.3mm_P2.50mm" H 3100 7200 50  0001 C CNN
 F 3 "~" H 3100 7200 50  0001 C CNN
 	1    3100 7200
@@
 	1    20300 1150
 	1    0    0    -1
-$EndComp
-$Comp
-L Device:R_Network08_US U8
-U 1 1 5E70F16A
-P 5700 2850
-F 0 "U8" V 5083 2850 50  0000 C CNN
-F 1 "4K7" V 5174 2850 50  0000 C CNN
-F 2 "Resistor_SMD:R_Array_Convex_5x1206" V 6175 2850 50  0001 C CNN
-F 3 "YC358TJK-074K7L" H 5700 2850 50  0001 C CNN
-	1    5700 2850
-	-1   0    0    1
-$EndComp
-$Comp
-L Device:R_Network08_US U12
-U 1 1 5E710830
-P 8750 2850
-F 0 "U12" V 8133 2850 50  0000 C CNN
-F 1 "4K7" V 8224 2850 50  0000 C CNN
-F 2 "Resistor_SMD:R_Array_Convex_5x1206" V 9225 2850 50  0001 C CNN
-F 3 "YC358TJK-074K7L" H 8750 2850 50  0001 C CNN
-	1    8750 2850
-	-1   0    0    1
-$EndComp
-$Comp
-L Device:R_Network08_US U15
-U 1 1 5E711DF2
-P 11500 2850
-F 0 "U15" V 10883 2850 50  0000 C CNN
-F 1 "4K7" V 10974 2850 50  0000 C CNN
-F 2 "Resistor_SMD:R_Array_Convex_5x1206" V 11975 2850 50  0001 C CNN
-F 3 "YC358TJK-074K7L" H 11500 2850 50  0001 C CNN
-	1    11500 2850
-	-1   0    0    1
 $EndComp
 $Comp
@@
 Wire Bus Line
 	16500 8950 16500 9150
-Wire Bus Line
-	14900 8950 12500 8950
 Connection ~ 12500 8950
 Wire Bus Line
@@
 P 16600 7750
 F 0 "U16" H 16800 7950 50  0000 C CNN
-F 1 "74LVC3G06" H 16900 7850 50  0000 C CNN
+F 1 "74LVC3G06DP" H 16900 7850 50  0000 C CNN
 F 2 "Package_SO:TSSOP-8_3x3mm_P0.65mm" H 16600 7750 50  0001 C CNN
 F 3 "http://www.ti.com/lit/sg/scyt129e/scyt129e.pdf" H 16600 7750 50  0001 C CNN
@@
 P 13100 7850
 F 0 "U16" H 13075 8117 50  0000 C CNN
-F 1 "74LVC3G06" H 13075 8026 50  0000 C CNN
+F 1 "74LVC3G06DP" H 13075 8026 50  0000 C CNN
 F 2 "Package_SO:TSSOP-8_3x3mm_P0.65mm" H 13100 7850 50  0001 C CNN
 F 3 "http://www.ti.com/lit/sg/scyt129e/scyt129e.pdf" H 13100 7850 50  0001 C CNN
@@
 P 16900 9500
 F 0 "U16" H 16875 9767 50  0000 C CNN
-F 1 "74LVC3G06" H 16875 9676 50  0000 C CNN
+F 1 "74LVC3G06DP" H 16875 9676 50  0000 C CNN
 F 2 "Package_SO:TSSOP-8_3x3mm_P0.65mm" H 16900 9500 50  0001 C CNN
 F 3 "http://www.ti.com/lit/sg/scyt129e/scyt129e.pdf" H 16900 9500 50  0001 C CNN
@@
 	3500 7300 3100 7300
 Connection ~ 3100 7300
+Wire Bus Line
+	12500 8950 15600 8950
+Connection ~ 15600 8950
+$Comp
+L 74xx:74LS74 U1
+U 3 1 5E69BE1C
+P 850 5750
+F 0 "U1" H 1080 5796 50  0000 L CNN
+F 1 "SN74LV74APWR" H 1080 5705 50  0000 L CNN
+F 2 "Package_SO:TSSOP-14_4.4x5mm_P0.65mm" H 850 5750 50  0001 C CNN
+F 3 "74xx/74hc_hct74.pdf" H 850 5750 50  0001 C CNN
+	3    850  5750
+	1    0    0    -1
+$EndComp
+$Comp
+L CPU2:R_Network08_US_YC358-TType U8
+U 1 1 5F45FDA7
+P 5700 2850
+F 0 "U8" H 5220 2804 50  0000 R CNN
+F 1 "4K7" H 5220 2895 50  0000 R CNN
+F 2 "Resistor_SMD:R_Array_Convex_5x1206" V 6175 2850 50  0001 C CNN
+F 3 "YC358TJK-074K7L" H 5700 2850 50  0001 C CNN
+	1    5700 2850
+	-1   0    0    1
+$EndComp
+$Comp
+L CPU2:R_Network08_US_YC358-TType U12
+U 1 1 5F466775
+P 8750 2850
+F 0 "U12" H 8270 2804 50  0000 R CNN
+F 1 "4K7" H 8270 2895 50  0000 R CNN
+F 2 "Resistor_SMD:R_Array_Convex_5x1206" V 9225 2850 50  0001 C CNN
+F 3 "YC358TJK-074K7L" H 8750 2850 50  0001 C CNN
+	1    8750 2850
+	-1   0    0    1
+$EndComp
+$Comp
+L CPU2:R_Network08_US_YC358-TType U15
+U 1 1 5F49ADAC
+P 11500 2850
+F 0 "U15" H 11020 2804 50  0000 R CNN
+F 1 "4K7" H 11020 2895 50  0000 R CNN
+F 2 "Resistor_SMD:R_Array_Convex_5x1206" V 11975 2850 50  0001 C CNN
+F 3 "YC358TJK-074K7L" H 11500 2850 50  0001 C CNN
+	1    11500 2850
+	-1   0    0    1
+$EndComp
+Wire Wire Line
+	6000 3050 6100 3050
+Connection ~ 6100 3050
+Wire Wire Line
+	9050 3050 9150 3050
+Connection ~ 9150 3050
+Wire Wire Line
+	11800 3050 11900 3050
+Connection ~ 11900 3050
 Wire Wire Line
 	19300 1400 20300 1400
