File: Commodore-64/c64-cpm-true/c64-cpm-true.sch (KiCad schematic (older format))
At the start: 51 parts, among them Q1 2N3906, U1 74S74, U10 74LS283, U11 74LS245, U12 4K7, U13 Z80CPU, U14 74LS245, U15 4K7, U2 74S04, U3 74LS367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

Commit message: Update to fit original CP/M case better
* Moved the left screwhole 0.5mm
* Moved the right screwhole 1mm
* Moved the top-right pinhole 0.2mm
* Removed the ground traces that went between card edge pads.
Connections:
- net ~ENCPM: now reaches C2.1, FB1.2, U2.1
Changed lines of the file:
@@
 	1900 3300 1900 3400
 Connection ~ 1900 3400
-Wire Wire Line
-	3700 2150 4100 2150
-Wire Wire Line
-	8350 2200 8800 2200
-Wire Wire Line
-	6000 2200 6450 2200
 $Comp
 L 74xx:74LS373 U4
@@
 	13100 1850 14150 1850
 Connection ~ 11000 550
-Wire Wire Line
-	13150 1150 14150 1150
 Connection ~ 12850 550
 Wire Bus Line
@@
 NoConn ~ 10150 10500
 Wire Wire Line
+	3700 2150 4100 2150
+Wire Wire Line
+	8350 2200 8800 2200
+Wire Wire Line
+	6000 2200 6450 2200
+Wire Wire Line
+	13150 1150 14150 1150
+Wire Bus Line
+	8750 4900 8750 5900
+Wire Bus Line
+	14800 7750 14800 8650
+Wire Bus Line
+	11100 8050 11100 8650
+Wire Bus Line
+	10850 7750 10850 7950
+Wire Bus Line
+	15900 7750 15900 9050
+Wire Wire Line
+	3700 1450 4100 1450
+Wire Wire Line
+	3700 1550 4100 1550
+Wire Wire Line
+	3700 1650 4100 1650
+Wire Wire Line
+	3700 1750 4100 1750
+Wire Wire Line
+	3700 1850 4100 1850
+Wire Wire Line
+	3700 1950 4100 1950
+Wire Wire Line
+	3700 2050 4100 2050
+Wire Wire Line
+	8350 1800 8800 1800
+Wire Wire Line
+	8350 1900 8800 1900
+Wire Wire Line
+	8350 2000 8800 2000
+Wire Wire Line
+	8350 2100 8800 2100
+Wire Wire Line
+	8350 1700 8800 1700
+Wire Wire Line
+	8350 1600 8800 1600
+Wire Wire Line
+	8350 1500 8800 1500
+Wire Wire Line
+	6000 1800 6450 1800
+Wire Wire Line
+	6000 1900 6450 1900
+Wire Wire Line
+	6000 2000 6450 2000
+Wire Wire Line
+	6000 2100 6450 2100
+Wire Wire Line
+	6000 1700 6450 1700
+Wire Wire Line
+	6000 1600 6450 1600
+Wire Wire Line
 	6000 1500 6450 1500
-Wire Wire Line
-	6000 1600 6450 1600
-Wire Wire Line
-	6000 1700 6450 1700
-Wire Wire Line
-	6000 2100 6450 2100
-Wire Wire Line
-	6000 2000 6450 2000
-Wire Wire Line
-	6000 1900 6450 1900
-Wire Wire Line
-	6000 1800 6450 1800
-Wire Wire Line
-	8350 1500 8800 1500
-Wire Wire Line
-	8350 1600 8800 1600
-Wire Wire Line
-	8350 1700 8800 1700
-Wire Wire Line
-	8350 2100 8800 2100
-Wire Wire Line
-	8350 2000 8800 2000
-Wire Wire Line
-	8350 1900 8800 1900
-Wire Wire Line
-	8350 1800 8800 1800
-Wire Wire Line
-	3700 2050 4100 2050
-Wire Wire Line
-	3700 1950 4100 1950
-Wire Wire Line
-	3700 1850 4100 1850
-Wire Wire Line
-	3700 1750 4100 1750
-Wire Wire Line
-	3700 1650 4100 1650
-Wire Wire Line
-	3700 1550 4100 1550
-Wire Wire Line
-	3700 1450 4100 1450
-Wire Bus Line
-	8750 4900 8750 5900
-Wire Bus Line
-	14800 7750 14800 8650
-Wire Bus Line
-	11100 8050 11100 8650
-Wire Bus Line
-	10850 7750 10850 7950
-Wire Bus Line
-	15900 7750 15900 9050
 Wire Bus Line
 	12850 550  12850 1350
@@
 Wire Bus Line
 	15900 550  15900 7750
+Text Label 11950 9050 0    50   ~ 0
+~ENCPM
 $EndSCHEMATC
